File: Production/Main Board - Double-Panel.brd (EAGLE design)
At the start: 138.2 x 176.3 mm, 210 parts, among them J1 MICROMOD-2222-C, J10 MICRO-SD-PUSH-PUSH-EXT-PIN, J12 Vertical Qwiic Connector, J14 QWIIC_RIGHT_ANGLE, J15 MICROMOD-2222-C, J18 CORTEX_JTAG_DEBUG_MINIMUM_PTH, J2 Vertical Qwiic Connector, J20 MICROMOD_CARRIER, J21 MICROMOD_CARRIER, J22 MICRO-SD-PUSH-PUSH-EXT-PIN, J4 QWIIC_RIGHT_ANGLE, J5 CORTEX_JTAG_DEBUG_MINIMUM_PTH, J6 MICROMOD_CARRIER, J7 MICROMOD_CARRIER, Q1 3.1A/30V/105mΩ, Q2 3.1A/30V/105mΩ, U1 MCP73831, U2 MCP73831, U3 AP7361C-33, U5 AP7361C-33

Commit message: Adds new panel that is a single column of three.
Parts:
- added 3V3_LED2, 5V_LED2: (no value), SparkFun-Jumpers:SMT-JUMPER_2_NC_TRACE_SILK
- added BYP2: JUMPER-SMT_2_NO_SILK, SparkFun-Jumpers:SMT-JUMPER_2_NO_SILK
- added C19, C20: 4.7uF, SparkFun-Capacitors:0603
- added C21, C25: 0.22uF, SparkFun-Capacitors:0603
- added C22, C24, C27: 0.1uF, SparkFun-Capacitors:0603
- added C23: 1.0uF, SparkFun-Capacitors:0603
- added C26: 10uF, SparkFun-Capacitors:0805
- added D11: Yellow, SparkFun-LED:LED-0603
- added D12: 3.3V, SparkFun-DiscreteSemi:SOD-323
- added D13, D15: RED, SparkFun-LED:LED-0603
- added D14: 3A/10V/280mV, SparkFun-DiscreteSemi:SOD-323
- added F3: 6V/2A, SparkFun-Fuses:1210
- added FD10, FD11, FD12, FD9: FIDUCIAL1X2, SparkFun-Aesthetics:FIDUCIAL-1X2
- added H19, H20, H25, H26: STAND-OFF-REFLOW-M2.5_2.5MM_TALL, SparkFun-Hardware:STAND-OFF-REFLOW-M2.5
- added H21, H22, H23, H24, H27: STAND-OFFTIGHT, SparkFun-Hardware:STAND-OFF-TIGHT
- added J25: Vertical Qwiic Connector, SparkFun-Connectors:JST04_1MM_VERT
- added J26: QWIIC_RIGHT_ANGLE, SparkFun-Connectors:JST04_1MM_RA
- added J27: MICROMOD-2222-C, SparkFun-MicroMod:M.2-CONNECTOR-E
- added J28: (no value), SparkFun-Connectors:JST-2-SMD
- added J29: (no value), SparkFun-Connectors:USB-C-16P-2LAYER-PADS
- added J30: CORTEX_JTAG_DEBUG_MINIMUM_PTH, SparkFun-Connectors:2X5-PTH-1.27MM
- added J31: (no value), SparkFun-Connectors:1X01_NO_SILK
- added J32, J33: MICROMOD_CARRIER, SparkFun-MicroMod-Function:M.2-CONNECTOR-E-FUNCTION-STANDARD
- added J34: MICRO-SD-PUSH-PUSH-EXT-PIN, SparkFun-Connectors:MICROSD-EXTERNALPIN
- added J35, J36: (no value), SparkFun-Connectors:1X03_LOCK
- added LOGO7: QWIIC_LOGO_8MM, SparkFun-Aesthetics:QWIIC_8MM
- added LOGO8: SFE_LOGO_NAME_FLAME.3_INCH, SparkFun-Aesthetics:SFE_LOGO_NAME_FLAME_.3
- added LOGO9: OSHW-LOGOL, SparkFun-Aesthetics:OSHW-LOGO-L
- added MEAS2: JUMPER-COMBO_2_NC_TRACE, SparkFun-Jumpers:COMBO-JUMPER_2_NC_TRACE
- added Q3: 3.1A/30V/105mΩ, SparkFun-DiscreteSemi:SOT23-3
- added R23, R27: 1k, SparkFun-Resistors:0603
- added R24, R25: 5.1k, SparkFun-Resistors:0603
- added R26: 100k, SparkFun-Resistors:0603
- added R28, R32, R33: 10k, SparkFun-Resistors:0603
- added R29: 20k, SparkFun-Resistors:0603
- added R30: 4.7k, SparkFun-Resistors:0603
- added R31: 2.0k, SparkFun-Resistors:0603
- added S7: Reset, SparkFun-Switches:TACTILE_SWITCH_SMD_5.2MM
- added S8: BOOT, SparkFun-Switches:TACTILE_SWITCH_SMD_5.2MM
- added S9: DIP-02-SMD-50MIL, SparkFun-Switches:DIPSWITCH-02-50MIL
- added TP10, TP11, TP12, TP9: TEST-POINT3X5, SparkFun-Connectors:PAD.03X.05
- added U$67: (no value), top:#3V3_EN#18
- added U$68: (no value), top:#3V3_LED#17
- added U$69: (no value), top:#VIN_LED#16
- added U$70: (no value), top:3V332533
- added U$71: (no value), top:VIN32532
- added U$72: (no value), top:CHG32531
- added U$73: (no value), top:#PTC#18
- added U$74: (no value), top:BOOT32541
- added U$75: (no value), top:RESET32540
- added U$76: (no value), top:PROCESSOR525
- added U$77: (no value), top:FUNCTION_ZERO520
- added U$78: (no value), top:FUNCTION_ONE524
- added U$79: (no value), SparkFun-MicroMod:MICROMOD_MI_LOGO_1
- added U$80: (no value), top:0523
- added U$81: (no value), top:1524
- added U$82: (no value), top:MAIN523
- added U$83: (no value), top:BOARD524
- added U$84: (no value), top:100MA6
- added U$85: (no value), top:500MA101
- added U$86: (no value), top:MAIN_BOARD5523
- added U$87: (no value), SparkFun-MicroMod:MICROMOD_LOGO_1
- added U$88: (no value), SparkFun-Aesthetics:QWIIC_3MM
- added U$89: (no value), top:STANDOFF501
- added U$90: (no value), SparkFun-Aesthetics:SFE_LOGO_FLAME_.3
- added U$91: (no value), top:#G6#517
- added U$92: (no value), top:#PWR_EN0#517
- added U$93: (no value), top:#PWR_EN1#517
- added U$94: (no value), top:#G5#517
- added U$95: (no value), top:#ALT_PWR_EN0#510
- added U$96: (no value), top:#ALT_PWR_EN1#510
- added U$97: (no value), top:#FC1#G3#518
- added U$98: (no value), top:#FC1#G4#518
- added U$99: (no value), top:#MEAS#40313513
- added U4: MCP73831, SparkFun-IC-Power:SOT23-5
- added U6: AP7361C-33, SparkFun-IC-Power:UDFN-8
- added VE2: (no value), SparkFun-Jumpers:SMT-JUMPER_2_NO_SILK
- moved E$3 73.6 mm to (127.1, 230.0)
- moved E$4 73.6 mm to (127.1, 230.0)
- moved E$1 73.6 mm to (-2.62, 230.0)
- moved E$2 73.6 mm to (-2.62, 230.0)
- moved E$5 15.3 mm to (-2.62, 6.35)
- moved E$6 15.3 mm to (-2.62, 6.35)
Connections:
- new net !BOOT!2: J27.11, S8.3, S8.4
- new net !CS0!-PROCESSOR2: J27.55, J32.49
- new net !CS1!-PROCESSOR2: J27.70, J33.49
- new net !RESET!2: J27.6, J30.10, J31.1, S7.3, S7.4
- new net 3.3V2: C23.1, C24.1, C25.1, C27.1, J25.2, J26.2, J27.2, J27.74, J30.1, J32.73, J33.36, J33.73, J34.4, MEAS2.2, MEAS2.4, R27.2, TP9.1
- new net 3.3V_EN2: J27.4, VE2.1
- new net 3.3V_EN_VE2: D12.C, R26.1, U6.5, VE2.2
- new net A0-PROCESSOR2: J27.34, J32.38
- new net A1-PROCESSOR2: J27.38, J33.38
- new net CTS1-PROCESSOR2: J27.15, J32.16
- new net D+2: J27.3, J29.A6, J29.B6
- new net D-2: J27.5, J29.A7, J29.B7
- new net D0-PROCESSOR2: J27.10, J32.47
- new net D1-PROCESSOR2: J27.18, J33.47
- new net G0-PROCESSOR2: J27.40, J32.53
- new net G1-PROCESSOR2: J27.42, J32.55
- new net G2-PROCESSOR2: J27.44, J32.57
- new net G3-PROCESSOR2: J27.46, J32.59
- new net G4-PROCESSOR/SD_CARD_!CS!2: J27.48, J32.61, J34.2
- new net G5-JUMPER2: J27.73, J35.2
- new net G5-PROCESSOR2: J33.53, J35.3
- new net G6-JUMPER2: J27.71, J36.2
- new net G6-PROCESSOR2: J33.55, J36.3
- new net G7-PROCESSOR2: J27.69, J33.57
- new net G8-PROCESSOR2: J27.62, J33.59
- new net G9-PROCESSOR2: J27.60, J33.61
- new net GND2: 3V3_LED2.1, 5V_LED2.1, C19.2, C20.2, C21.2, C22.2, C23.2, C24.2, C25.2, C26.2, C27.2, D12.A, H19.1, H20.1, H25.1, H26.1, J25.1, J26.1, J27.1, J27.33, J27.36, J27.39, J27.45, J27.7, J27.75, J28.1, J29.GND, J29.GND2, J30.3, J30.5, J30.9, J32.1, J32.32, J32.33, J32.34, J32.36, J32.39, J32.45, J32.75, J33.1, J33.32, J33.33, J33.34, J33.39, J33.45, J33.75, J34.10, J34.11, J34.12, J34.13, J34.6, R24.1, R25.1, R28.1, R31.1, R32.1, R33.1, S7.1, S7.2, S8.1, S8.2, U4.2, U6.4, U6.EP
- new net HOST_D+2: J27.35, J32.35
- new net HOST_D-2: J27.37, J32.37
- new net I2C_!INT!2: J27.16, J32.23, J33.23
- new net I2C_SCL2: J25.4, J26.4, J27.14, J32.21, J33.21
- new net I2C_SDA2: J25.3, J26.3, J27.12, J32.19, J33.19
- new net N$27: D11.C, R23.2
- new net N$28: R23.1, U4.1
- new net N$29: J29.B5, R25.2
- new net N$30: J29.A5, R24.2
- new net N$31: MEAS2.1, MEAS2.3, U6.1
- new net N$32: D13.A, R27.1
- new net N$33: BYP2.1, F3.1, J29.VBUS1, J29.VBUS2
- new net N$34: D15.A, R30.1
- new net N$35: 5V_LED2.2, D15.C
- new net N$36: 3V3_LED2.2, D13.C
- new net N$37: S9.3, S9.4, U4.5
- new net N$38: R31.2, S9.1
- new net N$39: R32.2, S9.2
- new net PROCESSOR_CAN-RX2: J27.41, J32.43
- new net PROCESSOR_CAN-TX2: J27.43, J32.41
- new net PWM0-PROCESSOR2: J27.32, J32.51
- new net PWM1-PROCESSOR2: J27.47, J33.51
- new net PWR_EN4: J27.68, J32.71, J35.1
- new net PWR_EN5: J27.66, J33.71, J36.1
- new net RTS1-PROCESSOR2: J27.13, J32.18
- new net RX1-PROCESSOR2: J27.19, J32.13
- new net RX2-PROCESSOR2: J27.20, J33.13
- new net SPI_PROCESSOR_SCK2: J27.57, J32.3, J33.3, J34.5
- new net SPI_PROCESSOR_SDI2: J27.61, J32.7, J33.7, J34.7
- new net SPI_PROCESSOR_SDO2: J27.59, J32.5, J33.5, J34.3
- new net SWDCK2: J27.21, J30.4
- new net SWDIO2: J27.23, J30.2, TP12.1
- new net TX1-PROCESSOR2: J27.17, J32.15
- new net TX2-PROCESSOR2: J27.22, J33.15
- new net VCC2: C19.1, C21.1, C22.1, C26.1, D11.A, D14.C, Q3.2, R26.2, U4.4, U6.8
- new net VIN/2: J27.49, R28.2, R29.1
- new net VIN2: BYP2.2, D14.A, F3.2, J27.9, J32.72, J32.74, J33.72, J33.74, Q3.1, R29.2, R30.2, R33.2, TP11.1
- new net V_BATT2: C20.1, J28.2, Q3.3, TP10.1, U4.3
Routing:
- net 3.3V2: track 0.00 -> 241.9 mm, vias 0 -> 11
- net VIN2: track 0.00 -> 179.2 mm, vias 0 -> 9
- net I2C_SCL2: track 0.00 -> 157.3 mm, vias 0 -> 8
- net I2C_SDA2: track 0.00 -> 156.1 mm, vias 0 -> 8
- net I2C_!INT!2: track 0.00 -> 153.2 mm, vias 0 -> 6
- net SPI_PROCESSOR_SDO2: track 0.00 -> 148.4 mm, vias 0 -> 4
- net SPI_PROCESSOR_SDI2: track 0.00 -> 143.5 mm, vias 0 -> 2
- net SPI_PROCESSOR_SCK2: track 0.00 -> 141.0 mm, vias 0 -> 2
- net PWR_EN5: track 0.00 -> 131.5 mm, vias 0 -> 5
- net !CS1!-PROCESSOR2: track 0.00 -> 124.9 mm, vias 0 -> 2
- net G8-PROCESSOR2: track 0.00 -> 122.8 mm, vias 0 -> 2
- net G9-PROCESSOR2: track 0.00 -> 120.6 mm, vias 0 -> 2
- net D0-PROCESSOR2: track 0.00 -> 111.7 mm, vias 0 -> 6
- net G5-PROCESSOR2: track 0.00 -> 111.6 mm, vias 0 -> 5
- net G4-PROCESSOR/SD_CARD_!CS!2: track 0.00 -> 109.0 mm, vias 0 -> 4
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- added copper zone on layer 1, net 3.3V2
- added copper zone on layer 1, net GND2
- added copper zone on layer 16, net GND2
- added copper zone on layer 1, net N$31
- added copper zone on layer 1, net N$33
- added copper zone on layer 1, net SHLD2
- added copper zone on layer 16, net SHLD2
- added copper zone on layer 1, net VCC2
- added copper zone on layer 1, net VIN2
Other:
- board size 138.2 x 176.3 mm -> 138.2 x 254 mm

Commit message: Updates panel
Connections:
- net VCC: now also J6.72, J6.74, J7.72, J7.74
- net VCC1: now also J20.72, J20.74, J21.72, J21.74
- net VCC2: now also J32.72, J32.74, J33.72, J33.74
- net VIN: no longer J6.72, J6.74, J7.72, J7.74
- net VIN1: no longer J20.72, J20.74, J21.72, J21.74
- net VIN2: no longer J32.72, J32.74, J33.72, J33.74
Routing:
- net VCC: track 55.5 -> 156.4 mm, vias 2 -> 5
- net VCC2: track 55.5 -> 156.4 mm, vias 2 -> 5
- net VCC1: track 55.5 -> 156.4 mm, vias 2 -> 5
- net VIN: track 179.2 -> 81.6 mm, vias 9 -> 3
- net VIN2: track 179.2 -> 81.6 mm, vias 9 -> 3
- net VIN1: track 179.2 -> 81.6 mm, vias 9 -> 3
- net GND2: vias 82 -> 84
- net GND1: vias 82 -> 84
- net GND: vias 82 -> 84
Other:
- board text added: "v11"
- board text removed: "v10"
