File: Production/SparkFun_Main_Board_Double_v22-Panel.brd (EAGLE design)
At the start: 124.5 x 73.7 mm, 134 parts, among them J1 MICROMOD-2222-C, J10 MICRO-SD-PUSH-PUSH-EXT-PIN, J2 Vertical Qwiic Connector, J4 QWIIC_RIGHT_ANGLE, J5 CORTEX_JTAG_DEBUG_MINIMUM_PTH, J6 MICROMOD_FUNCTION_MAIN, J7 MICROMOD_FUNCTION_MAIN, Q1 3.1A/30V/105mΩ, Q2 20V/4.2A/52mΩ/1.4W, U1 STG3856QTR, U2 MCP73831, U3 ESD Diode, U4 AP7347DQ-33W5-7K-3.3V, U5 AP7361C-33

Commit message: Adds new production files
Parts:
- removed FRAME1: FRAME-LEDGER, SparkFun-Aesthetics:CREATIVE_COMMONS
- removed FRAME2: FRAME-LEDGERNO_FOOTPRINT, SparkFun-Aesthetics:DUMMY
- added 3V3_LED1, 3V3_LED2, 5V_LED1, 5V_LED2, DIVIDER1, DIVIDER2, QWIIC_LED1, QWIIC_LED2, SHLD1, SHLD2: JUMPER-SMT_2_NC_TRACE_SILK, SparkFun-Jumpers:SMT-JUMPER_2_NC_TRACE_SILK
- added 3V3_MEAS1, 3V3_MEAS2, 5V_MEAS1, 5V_MEAS2: JUMPER-COMBO_2_NC_TRACE, SparkFun-Jumpers:COMBO-JUMPER_2_NC_TRACE
- added BYP1, BYP2, VE1, VE2: JUMPER-SMT_2_NO_SILK, SparkFun-Jumpers:SMT-JUMPER_2_NO_SILK
- added C10, C13, C19, C20, C22, C9: 4.7uF, SparkFun-Capacitors:0603
- added C12, C21: 0.1uF, SparkFun-Capacitors:0603
- added C14, C17, C23, C26: 10uF, SparkFun-Capacitors:0805
- added C15, C16, C24, C25: 1.0uF, SparkFun-Capacitors:0603
- added C18, C27: 10uF, SparkFun-Capacitors:0603
- added D10, D16: 3A/40V/500mV, SparkFun-DiscreteSemi:SMA-DIODE
- added D11, D12, D15, D17, D18, D9: RED, SparkFun-LED:LED-0603
- added D13, D6: Yellow, SparkFun-LED:LED-0603
- added D14, D7: 3.3V, SparkFun-DiscreteSemi:SOD-323
- added E$1, E$2, E$3, E$4: (no value), SparkFun-Aesthetics:FIDUCIAL-1X2
- added E$5, E$6: (no value), SparkFun-Retired:FIDUCIAL-1.5X3
- added F1, F3: 6V/2A, SparkFun-Fuses:1210
- added FD10, FD11, FD12, FD5, FD6, FD7, FD8, FD9: FIDUCIAL1X2, SparkFun-Aesthetics:FIDUCIAL-1X2
- added H10, H11, H18, H21, H22, H23, H24, H27, H7, H9: STAND-OFFTIGHT, SparkFun-Hardware:STAND-OFF-TIGHT
- added H12, H13, H19, H20, H25, H26, H5, H6: STAND-OFF-REFLOW-M2.5_2.5MM_TALL, SparkFun-Hardware:STAND-OFF-REFLOW-M2.5
- added I2C_PU1, I2C_PU2: JUMPER-SMT_3_2-NC_TRACE_SILK, SparkFun-Jumpers:SMT-JUMPER_3_2-NC_TRACE_SILK
- added J12, J25: Vertical Qwiic Connector, SparkFun-Connectors:JST04_1MM_VERT
- added J14, J26: QWIIC_RIGHT_ANGLE, SparkFun-Connectors:JST04_1MM_RA
- added J15, J27: MICROMOD-2222-C, SparkFun-MicroMod:M.2-CONNECTOR-E
- added J16, J28: (no value), SparkFun-Connectors:JST-2-SMD
- added J17, J29: (no value), SparkFun-Connectors:USB-C-16P-2LAYER-PADS
- added J18, J30: CORTEX_JTAG_DEBUG_MINIMUM_PTH, SparkFun-Connectors:2X5-PTH-1.27MM
- added J19, J23, J31, J35: (no value), SparkFun-Connectors:1X01_NO_SILK
- added J20, J32: MICRO-SD-PUSH-PUSH-EXT-PIN, SparkFun-Connectors:MICROSD-EXTERNALPIN
- added J21, J22, J33, J34: MICROMOD_FUNCTION_MAIN, SparkFun-MicroMod:M.2-CONNECTOR-E-FUNCTION-STANDARD
- added J24, J36: (no value), SparkFun-Connectors:1X02_NO_SILK
- added LOGO4, LOGO7: QWIIC_LOGO_8MM, SparkFun-Aesthetics:QWIIC_8MM
- added LOGO5, LOGO8: SFE_LOGO_NAME_FLAME.3_INCH, SparkFun-Aesthetics:SFE_LOGO_NAME_FLAME_.3
- added LOGO6, LOGO9: OSHW-LOGOL, SparkFun-Aesthetics:OSHW-LOGO-L
- added Q3, Q5: 3.1A/30V/105mΩ, SparkFun-DiscreteSemi:SOT23-3
- added Q4, Q6: 20V/4.2A/52mΩ/1.4W, SparkFun-DiscreteSemi:SOT23-3
- added R17, R37: 4.7k, SparkFun-Resistors:0603
- added R20, R21, R38, R39: 5.1k, SparkFun-Resistors:0603
- added R22, R29, R30, R33, R36, R40, R47, R48, R51, R54: 100k, SparkFun-Resistors:0603
- added R23, R34, R41, R52: 1k, SparkFun-Resistors:0603
- added R24, R28, R42, R46: 10k, SparkFun-Resistors:0603
- added R25, R43: 20k, SparkFun-Resistors:0603
- added R26, R31, R32, R44, R49, R50: 2.2k, SparkFun-Resistors:0603
- added R27, R45: 2.0k, SparkFun-Resistors:0603
- added R35, R53: 100, SparkFun-Resistors:0603
- added S10, S13, S14, S15, S6, S9: (no value), SparkFun-Switches:SWITCH_SPST_SMD_A
- added S11, S4: Reset, SparkFun-Switches:TACTILE_SWITCH_SMD_5.2MM
- added S12, S5: BOOT, SparkFun-Switches:TACTILE_SWITCH_SMD_5.2MM
- added TP10, TP11, TP12, TP5, TP6, TP7, TP8, TP9: TEST-POINT3X5, SparkFun-Connectors:PAD.03X.05
- added U$100, U$54: (no value), top:FUNCTION_ONE524
- added U$101, U$55: (no value), SparkFun-MicroMod:MICROMOD_MI_LOGO_1
- added U$102, U$56: (no value), top:0523
- added U$103, U$57: (no value), top:1524
- added U$104, U$58: (no value), top:MAIN523
- added U$105, U$59: (no value), top:BOARD524
- added U$106, U$60: (no value), top:MAIN_BOARD5523
- added U$107, U$61: (no value), SparkFun-MicroMod:MICROMOD_LOGO_1
- added U$108, U$62: (no value), SparkFun-Aesthetics:QWIIC_3MM
- added U$109, U$63: (no value), top:STANDOFF501
- added U$110, U$64: (no value), SparkFun-Aesthetics:SFE_LOGO_FLAME_.3
- added U$111, U$65: (no value), top:#CS_ALT#20
- added U$112, U$66: (no value), top:#CS_DEF#19
- added U$113, U$67: (no value), top:#G5_PROC#21
- added U$114, U$68: (no value), top:#G6_PROC#21
- added U$115, U$69: (no value), top:#EN0_ALT#21
- added U$116, U$70: (no value), top:#EN1_ALT#21
- added U$117, U$71: (no value), top:CHARGE501
- added U$118, U$72: (no value), top:#SHLD#501
- added U$119, U$73: (no value), top:#I2C#501
- added U$120, U$74: (no value), top:#3V3_MEAS#6522
- added U$121, U$75: (no value), top:#5V_MEAS#6522
- added U$122, U$76: (no value), top:500MA6520
- added U$123, U$77: (no value), top:G518
- added U$124, U$78: (no value), top:G6519
- added U$125, U$79: (no value), top:CS17
- added U$126, U$80: (no value), top:SWD6522
- added U$127, U$81: (no value), top:#3V3_EN#23
- added U$128, U$82: (no value), top:#3V3_LED#22
- added U$129, U$83: (no value), top:#QWIIC_LED#22
- added U$130, U$84: (no value), top:#DIVIDER#23
- added U$131, U$85: (no value), top:#VIN_LED#24
- added U$132, U$86: (no value), top:QWC18
- added U$133, U$87: (no value), SparkFun-Aesthetics:SFE_LOGO_NAME_FLAME_.1
- added U$134, U$88: (no value), top:#PTC#13
- added U$135, U$3, U$89: (no value), top:##RST##8
- added U$136, U$137, U$90, U$91: (no value), top:#GND#10
- added U$138, U$46, U$92: (no value), top:#VBAT#9
- added U$47, U$93: (no value), top:3V332533
- added U$48, U$94: (no value), top:VIN32532
- added U$49, U$95: (no value), top:CHG32531
- added U$50, U$96: (no value), top:BOOT32541
- added U$51, U$97: (no value), top:RESET32540
- added U$52, U$98: (no value), top:PROCESSOR525
- added U$53, U$99: (no value), top:FUNCTION_ZERO520
- added U10, U15: AP7347DQ-33W5-7K-3.3V, dip_switch:SOT25
- added U11, U6: MCP73831, SparkFun-IC-Power:SOT23-5
- added U12, U7: AP7361C-33, SparkFun-IC-Power:UDFN-8
- added U13, U8: STG3856QTR, dip_switch:STG3856
- added U14, U9: ESD Diode, SparkFun-DiscreteSemi:SOT-23-6
- U$39: device top:#RST#6521 -> top:#GND#10
- U$40: device top:#GND#6520 -> top:#GND#10
- moved U$33 12.3 mm to (109.2, 3.56)
- moved J11 11.8 mm to (118.7, 8.38)
- moved TP3 10.2 mm to (106.7, 5.08)
- moved U$40 10.0 mm to (120.9, 8.38), turned to 0 degrees
- moved U$27 5.71 mm to (115.6, 3.56)
- moved C4 4.80 mm to (110.5, 16.6), turned to 90 degrees
- moved J8 2.84 mm to (111.8, 7.62), turned to 180 degrees
- moved U$39 2.54 mm to (119.4, 18.3)
- moved U$14 1.52 mm to (106.8, 16.4)
- moved C3 1.40 mm to (116.8, 16.6)
- moved R7 1.27 mm to (113.4, 22.2)
- moved R10 1.27 mm to (113.4, 20.7)
- moved R3 1.27 mm to (113.4, 19.2)
- moved U2 1.27 mm to (113.4, 16.6)
- moved U$25 0.73 mm to (119.5, 13.0)
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Connections:
- new net !BOOT!1: J15.11, J21.66, J22.66, S5.3, S5.4
- new net !BOOT!2: J27.11, J33.66, J34.66, S12.3, S12.4
- new net !CS0!-PROCESSOR1: J15.55, J21.49
- new net !CS0!-PROCESSOR2: J27.55, J33.49
- new net !CS1!-PROC-JUMPER1: J22.49, S10.2
- new net !CS1!-PROC-JUMPER2: J34.49, S15.2
- new net !CS1!-PROCESSOR1: J15.70, S10.1
- new net !CS1!-PROCESSOR2: J27.70, S15.1
- new net !DFU-FC0!1: J21.10, R30.2, U8.P12
- new net !DFU-FC0!2: J33.10, R48.2, U13.P12
- new net !DFU-FC1!1: J22.10, R29.1, U8.P10
- new net !DFU-FC1!2: J34.10, R47.1, U13.P10
- new net !RESET!1: J15.6, J18.10, J19.1, J21.68, J22.68, S4.3, S4.4
- new net !RESET!2: J27.6, J30.10, J31.1, J33.68, J34.68, S11.3, S11.4
- new net 3.3V1: 3V3_MEAS1.2, 3V3_MEAS1.4, I2C_PU1.2, J15.2, J15.74, J18.1, J21.73, J22.36, J22.73, Q4.2, R23.2, R29.2, R30.1, TP5.1, U8.P11
- new net 3.3V2: 3V3_MEAS2.2, 3V3_MEAS2.4, I2C_PU2.2, J27.2, J27.74, J30.1, J33.73, J34.36, J34.73, Q6.2, R41.2, R47.2, R48.1, TP9.1, U13.P11
- new net 3.3V_EN1: J15.4, VE1.1
- new net 3.3V_EN2: J27.4, VE2.1
- new net 3.3V_EN_VE1: D7.C, R22.1, U7.5, VE1.2
- new net 3.3V_EN_VE2: D14.C, R40.1, U12.5, VE2.2
- new net 3.3V_QWIIC1: C15.1, J12.2, J14.2, R34.2, U10.5
- new net 3.3V_QWIIC2: C24.1, J25.2, J26.2, R52.2, U15.5
- new net 3V3_MEAS1: 3V3_MEAS1.1, 3V3_MEAS1.3, C13.1, C17.1, U7.1
- new net 3V3_MEAS2: 3V3_MEAS2.1, 3V3_MEAS2.3, C22.1, C26.1, U12.1
- new net 5V_MEAS1: 5V_MEAS1.2, 5V_MEAS1.4, C12.1, C14.1, R22.2, U7.8
- new net 5V_MEAS2: 5V_MEAS2.2, 5V_MEAS2.4, C21.1, C23.1, R40.2, U12.8
- new net A0-PROCESSOR1: J15.34, J21.38
- new net A0-PROCESSOR2: J27.34, J33.38
- new net A1-PROCESSOR/!CS1!-ALT1: J15.38, J22.38, S10.3
- new net A1-PROCESSOR/!CS1!-ALT2: J27.38, J34.38, S15.3
- new net CTS1-PROCESSOR1: J15.15, J21.16
- new net CTS1-PROCESSOR2: J27.15, J33.16
- new net D+1: J15.3, J17.A6, J17.B6, U9.6
- new net D+2: J27.3, J29.A6, J29.B6, U14.6
- new net D-1: J15.5, J17.A7, J17.B7, U9.4
- new net D-2: J27.5, J29.A7, J29.B7, U14.4
- new net D0-PROCESSOR1: J15.10, J21.47
- new net D0-PROCESSOR2: J27.10, J33.47
- new net D1-PROCESSOR1: J15.18, J22.47
- new net D1-PROCESSOR2: J27.18, J34.47
- new net G0-PROCESSOR1: J15.40, J21.53
- new net G0-PROCESSOR2: J27.40, J33.53
- new net G1-PROCESSOR1: J15.42, J21.55
- new net G1-PROCESSOR2: J27.42, J33.55
- new net G2-PROCESSOR1: J15.44, J21.57
- new net G2-PROCESSOR2: J27.44, J33.57
- new net G3-PROCESSOR1: J15.46, J21.59
- new net G3-PROCESSOR2: J27.46, J33.59
- new net G4-PROCESSOR/SD_CARD_!CS!1: J15.48, J20.2, J21.61
- new net G4-PROCESSOR/SD_CARD_!CS!2: J27.48, J32.2, J33.61
- new net G5-JUMPER1: J15.73, S6.2
- new net G5-JUMPER2: J27.73, S13.2
- new net G5-PROCESSOR1: J22.53, S6.1
- new net G5-PROCESSOR2: J34.53, S13.1
- new net G6-JUMPER1: J15.71, S9.2
- new net G6-JUMPER2: J27.71, S14.2
- new net G6-PROCESSOR1: J22.55, S9.1
- new net G6-PROCESSOR2: J34.55, S14.1
- new net G7-PROCESSOR1: J15.69, J22.57
- new net G7-PROCESSOR2: J27.69, J34.57
- new net GND1: 3V3_LED1.1, 5V_LED1.1, C10.2, C12.2, C13.2, C14.2, C15.2, C16.2, C17.2, C18.1, C9.2, D7.A, DIVIDER1.1, H12.1, H13.1, H5.1, H6.1, J12.1, J14.1, J15.1, J15.33, J15.36, J15.39, J15.45, J15.7, J15.75, J16.1, J17.GND, J17.GND2, J18.3, J18.5, J18.9, J20.10, J20.11, J20.12, J20.13, J20.6, J21.1, J21.2, J21.32, J21.33, J21.34, J21.36, J21.39, J21.45, J21.75, J21.8, J22.1, J22.2, J22.32, J22.33, J22.34, J22.39, J22.45, J22.75, J22.8, J23.1, J24.1, QWIIC_LED1.1, R20.1, R21.1, R27.1, R28.1, R36.2, S4.1, S4.2, S5.1, S5.2, SHLD1.1, U10.2, U6.2, U7.4, U7.EP, U8.P5, U9.2
- new net GND2: 3V3_LED2.1, 5V_LED2.1, C19.2, C20.2, C21.2, C22.2, C23.2, C24.2, C25.2, C26.2, C27.1, D14.A, DIVIDER2.1, H19.1, H20.1, H25.1, H26.1, J25.1, J26.1, J27.1, J27.33, J27.36, J27.39, J27.45, J27.7, J27.75, J28.1, J29.GND, J29.GND2, J30.3, J30.5, J30.9, J32.10, J32.11, J32.12, J32.13, J32.6, J33.1, J33.2, J33.32, J33.33, J33.34, J33.36, J33.39, J33.45, J33.75, J33.8, J34.1, J34.2, J34.32, J34.33, J34.34, J34.39, J34.45, J34.75, J34.8, J35.1, J36.1, QWIIC_LED2.1, R38.1, R39.1, R45.1, R46.1, R54.2, S11.1, S11.2, S12.1, S12.2, SHLD2.1, U11.2, U12.4, U12.EP, U13.P5, U14.2, U15.2
- new net HOST_D+1: J15.35, J21.35
- new net HOST_D+2: J27.35, J33.35
- new net HOST_D-1: J15.37, J21.37
- new net HOST_D-2: J27.37, J33.37
- new net I2C_!INT!1: J15.16, J21.23, J22.23
- new net I2C_!INT!2: J27.16, J33.23, J34.23
- new net I2C_SCL1: J12.4, J14.4, J15.14, J21.21, J22.21, R32.1
- new net I2C_SCL1-PROCESSOR/QWIIC_EN1: J15.53, R33.1, U10.3
- new net I2C_SCL1-PROCESSOR/QWIIC_EN2: J27.53, R51.1, U15.3
- new net I2C_SCL2: J25.4, J26.4, J27.14, J33.21, J34.21, R50.1
- new net I2C_SDA1: J12.3, J14.3, J15.12, J21.19, J22.19, R31.1
- new net I2C_SDA1-PROCESSOR/!SD_ENABLE!1: J15.51, R35.1
- new net I2C_SDA1-PROCESSOR/!SD_ENABLE!2: J27.51, R53.1
- new net I2C_SDA2: J25.3, J26.3, J27.12, J33.19, J34.19, R49.1
- new net N$15: D6.C, U6.1
- new net N$17: J17.B5, R21.2
- new net N$19: J17.A5, R20.2
- new net N$20: D9.A, R23.1
- new net N$21: D11.A, R26.1
- new net N$22: 5V_LED1.2, D11.C
- new net N$23: 3V3_LED1.2, D9.C
- new net N$24: I2C_PU1.3, R31.2
- new net N$25: I2C_PU1.1, R32.2
- new net N$26: R27.2, U6.5
- new net N$27: DIVIDER1.2, R24.1
- new net N$28: D12.C, QWIIC_LED1.2
- new net N$29: D12.A, R34.1
- new net N$30: C18.2, J20.4, Q4.3
- new net N$31: Q4.1, R35.2, R36.1
- new net N$32: D6.A, R17.2
- new net N$33: D13.C, U11.1
- new net N$34: J29.B5, R39.2
- new net N$35: J29.A5, R38.2
- new net N$36: D15.A, R41.1
- new net N$37: D17.A, R44.1
- new net N$38: 5V_LED2.2, D17.C
- new net N$39: 3V3_LED2.2, D15.C
- new net N$40: I2C_PU2.3, R49.2
- new net N$41: I2C_PU2.1, R50.2
- new net N$42: R45.2, U11.5
- new net N$43: DIVIDER2.2, R42.1
- new net N$44: D18.C, QWIIC_LED2.2
- new net N$45: D18.A, R52.1
- new net N$46: C27.2, J32.4, Q6.3
- new net N$47: Q6.1, R53.2, R54.1
- new net N$48: D13.A, R37.2
- new net PROCESSOR_CAN-RX1: J15.41, J21.43
- new net PROCESSOR_CAN-RX2: J27.41, J33.43
- new net PROCESSOR_CAN-TX1: J15.43, J21.41
- new net PROCESSOR_CAN-TX2: J27.43, J33.41
- new net PWM0-PROCESSOR1: J15.32, J21.51
- new net PWM0-PROCESSOR2: J27.32, J33.51
- new net PWM1-PROCESSOR1: J15.47, J22.51
- new net PWM1-PROCESSOR2: J27.47, J34.51
- new net RTS1-PROCESSOR1: J15.13, J21.18
- new net RTS1-PROCESSOR2: J27.13, J33.18
- new net RX1-DFU_TX-FC0-PLEX1: J21.4, U8.P9
- new net RX1-DFU_TX-FC0-PLEX2: J33.4, U13.P9
- new net RX1-DFU_TX-FC1-PLEX1: J22.4, U8.P8
- new net RX1-DFU_TX-FC1-PLEX2: J34.4, U13.P8
- new net RX1-PROCESSOR-PLEX1: J21.13, U8.P7
- new net RX1-PROCESSOR-PLEX2: J33.13, U13.P7
- new net RX1-PROCESSOR1: J15.19, U8.P6
- new net RX1-PROCESSOR2: J27.19, U13.P6
- new net RX2-PROCESSOR1: J15.20, J22.13
- new net RX2-PROCESSOR2: J27.20, J34.13
- new net SDIO_DATA1/PWR_EN1_ALT1: J15.66, J22.71, S9.3
- new net SDIO_DATA1/PWR_EN1_ALT2: J27.66, J34.71, S14.3
- new net SDIO_DATA2/PWR_EN0_ALT1: J15.68, J21.71, S6.3
- new net SDIO_DATA2/PWR_EN0_ALT2: J27.68, J33.71, S13.3
- new net SHLD1: J17.SHLD1, J17.SHLD2, J17.SHLD3, J17.SHLD4, SHLD1.2
- new net SHLD2: J29.SHLD1, J29.SHLD2, J29.SHLD3, J29.SHLD4, SHLD2.2
- new net SPI_PROCESSOR_SCK1: J15.57, J20.5, J21.3, J22.3
- new net SPI_PROCESSOR_SCK2: J27.57, J32.5, J33.3, J34.3
- new net SPI_PROCESSOR_SDI1: J15.61, J20.7, J21.7, J22.7
- new net SPI_PROCESSOR_SDI2: J27.61, J32.7, J33.7, J34.7
- new net SPI_PROCESSOR_SDO1: J15.59, J20.3, J21.5, J22.5
- new net SPI_PROCESSOR_SDO2: J27.59, J32.3, J33.5, J34.5
- new net SPI_SCK1-PROCESSOR1: J15.60, J22.61
- new net SPI_SCK1-PROCESSOR2: J27.60, J34.61
- new net SPI_SDO1-PROCESSOR1: J15.62, J22.59
- new net SPI_SDO1-PROCESSOR2: J27.62, J34.59
- new net SWDCK1: J15.21, J18.4
- new net SWDCK2: J27.21, J30.4
- new net SWDIO1: J15.23, J18.2, TP8.1
- new net SWDIO2: J27.23, J30.2, TP12.1
- new net TX1-DFU_RX-FC0-PLEX1: J21.6, U8.P1
- new net TX1-DFU_RX-FC0-PLEX2: J33.6, U13.P1
- new net TX1-DFU_RX-FC1-PLEX1: J22.6, U8.P2
- new net TX1-DFU_RX-FC1-PLEX2: J34.6, U13.P2
- new net TX1-PROCESSOR-PLEX1: J21.15, U8.P3
- new net TX1-PROCESSOR-PLEX2: J33.15, U13.P3
- new net TX1-PROCESSOR1: J15.17, U8.P4
- new net TX1-PROCESSOR2: J27.17, U13.P4
- new net TX2-PROCESSOR1: J15.22, J22.15
- new net TX2-PROCESSOR2: J27.22, J34.15
- new net VCC1: 5V_MEAS1.1, 5V_MEAS1.3, C16.1, D10.C, J21.72, J21.74, J22.72, J22.74, Q3.2, R33.2, U10.1
- new net VCC2: 5V_MEAS2.1, 5V_MEAS2.3, C25.1, D16.C, J33.72, J33.74, J34.72, J34.74, Q5.2, R51.2, U15.1
- new net VIN/1: J15.49, R24.2, R25.1
- new net VIN/2: J27.49, R42.2, R43.1
- new net VIN1: BYP1.2, C9.1, D10.A, F1.2, J15.9, Q3.1, R17.1, R25.2, R26.2, R28.2, TP7.1, U6.4
- new net VIN2: BYP2.2, C19.1, D16.A, F3.2, J27.9, Q5.1, R37.1, R43.2, R44.2, R46.2, TP11.1, U11.4
- new net V_BATT1: C10.1, J16.2, J24.2, Q3.3, TP6.1, U6.3
- new net V_BATT2: C20.1, J28.2, J36.2, Q5.3, TP10.1, U11.3
- new net V_USB1: BYP1.1, F1.1, J17.VBUS1, J17.VBUS2, U9.5
- new net V_USB2: BYP2.1, F3.1, J29.VBUS1, J29.VBUS2, U14.5
- net !CS1!-PROC-JUMPER: now also J7.49; no longer J7.38
- net !CS1!-PROCESSOR: no longer J7.49
- net A1-PROCESSOR/!CS1!-ALT: now also J7.38
Routing:
- net 3.3V2: track 0.00 -> 237.7 mm, vias 0 -> 21
- net 3.3V1: track 0.00 -> 237.7 mm, vias 0 -> 21
- net VCC1: track 0.00 -> 168.9 mm, vias 0 -> 9
- net VCC2: track 0.00 -> 168.9 mm, vias 0 -> 9
- net I2C_!INT!2: track 0.00 -> 164.3 mm, vias 0 -> 6
- net I2C_!INT!1: track 0.00 -> 164.3 mm, vias 0 -> 6
- net SPI_PROCESSOR_SDO2: track 0.00 -> 158.9 mm, vias 0 -> 4
- net SPI_PROCESSOR_SDO1: track 0.00 -> 158.9 mm, vias 0 -> 4
- net I2C_SDA1: track 0.00 -> 158.5 mm, vias 0 -> 8
- net I2C_SDA2: track 0.00 -> 158.5 mm, vias 0 -> 8
- net SPI_PROCESSOR_SCK2: track 0.00 -> 157.3 mm, vias 0 -> 4
- net SPI_PROCESSOR_SCK1: track 0.00 -> 157.3 mm, vias 0 -> 4
- net I2C_SCL2: track 0.00 -> 156.7 mm, vias 0 -> 7
- net I2C_SCL1: track 0.00 -> 156.7 mm, vias 0 -> 7
- net !RESET!1: track 0.00 -> 154.4 mm, vias 0 -> 6
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- added copper zone on layer 1, net 3.3V1
- added copper zone on layer 1, net 3.3V2
- added copper zone on layer 1, net 3V3_MEAS1
- added copper zone on layer 1, net 3V3_MEAS2
- added copper zone on layer 1, net 5V_MEAS1
- added copper zone on layer 1, net 5V_MEAS2
- added copper zone on layer 1, net GND1
- added copper zone on layer 16, net GND1
- added copper zone on layer 1, net GND2
- added copper zone on layer 16, net GND2
- added copper zone on layer 1, net SHLD1
- added copper zone on layer 16, net SHLD1
- added copper zone on layer 1, net SHLD2
- added copper zone on layer 16, net SHLD2
- added copper zone on layer 1, net VCC1
- added copper zone on layer 1, net VCC2
- added copper zone on layer 1, net VIN1
- added copper zone on layer 1, net VIN2
- added copper zone on layer 1, net V_USB1
- added copper zone on layer 1, net V_USB2
Other:
- board size 124.5 x 73.7 mm -> 138.2 x 254 mm
- board text added: "Route Out"
- board text added: "v-score"
- board text added: "v22"
- board text removed: "Elias Santistevan"
- board text removed: "Units in Inches"
- board text removed: "v21"
