File: Hardware/Discrete/Main Board - Double _Discrete.brd (EAGLE design)
At the start: 124.5 x 73.7 mm, 127 parts, among them J1 MICROMOD-2222-C, J10 MICRO-SD-PUSH-PUSH-EXT-PIN, J2 Vertical Qwiic Connector, J4 QWIIC_RIGHT_ANGLE, J5 CORTEX_JTAG_DEBUG_MINIMUM_PTH, J6 MICROMOD_FUNCTION_MAIN, J7 MICROMOD_FUNCTION_MAIN, Q1 3.1A/30V/105mΩ, U1 SN74HCS4075PWR, U2 MCP73831, U3 ESD Diode, U4 AP7347DQ-33W5-7K-3.3V, U5 AP7361C-33, U6 74HC2G04GV, U7 SN74HCS11PWR, U8 SN74HCS4075PWR

Commit message: Matches length of D+ and D-
Parts:
- U1: value SN74HCS4075PWR -> SN74HCS11PWR
Connections:
- new net N$16: U7.P2
- new net N$17: U7.P13
- new net N$18: U7.P3
- new net N$19: U7.P4
- new net N$20: U7.P5
- new net N$21: U7.P9
- new net N$22: U7.P10
- new net N$23: U7.P11
- new net N$9: U7.P1
Changed lines of the file:
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@@
 <attribute name="VALUE" x="-29.21" y="-37.592" size="0.6096" layer="27" font="vector" ratio="20" align="top-center"/>
 </element>
-<element name="U1" library="dip_switch" package="TSSOP14" value="SN74HCS4075PWR" x="-27.94" y="-43.18" smashed="yes">
+<element name="U1" library="dip_switch" package="TSSOP14" value="SN74HCS11PWR" x="-27.94" y="-43.18" smashed="yes">
 <attribute name="NAME" x="-29.337" y="-40.386" size="0.6096" layer="25" font="vector" ratio="20"/>
 <attribute name="PROD_ID" value="" x="-35.56" y="-34.29" size="1.778" layer="27" font="vector" ratio="15" display="off"/>
@@
 <contactref element="U6" pad="P3"/>
 </signal>
+<signal name="N$9">
+<contactref element="U7" pad="P1"/>
+</signal>
+<signal name="N$16">
+<contactref element="U7" pad="P2"/>
+</signal>
+<signal name="N$17">
+<contactref element="U7" pad="P13"/>
+</signal>
+<signal name="N$18">
+<contactref element="U7" pad="P3"/>
+</signal>
+<signal name="N$19">
+<contactref element="U7" pad="P4"/>
+</signal>
+<signal name="N$20">
+<contactref element="U7" pad="P5"/>
+</signal>
+<signal name="N$21">
+<contactref element="U7" pad="P9"/>
+</signal>
+<signal name="N$22">
+<contactref element="U7" pad="P10"/>
+</signal>
+<signal name="N$23">
+<contactref element="U7" pad="P11"/>
+</signal>
 </signals>
