File: Hardware/Main Board - Double v3.brd (EAGLE design)
At the start: 124.5 x 73.7 mm, 134 parts, among them J1 MICROMOD-2222-C, J10 MICRO-SD-PUSH-PUSH-EXT-PIN, J2 Vertical Qwiic Connector, J4 QWIIC_RIGHT_ANGLE, J5 CORTEX_JTAG_DEBUG_MINIMUM_PTH, J6 MICROMOD_FUNCTION_MAIN, J7 MICROMOD_FUNCTION_MAIN, Q1 3.1A/30V/105mΩ, Q2 20V/4.2A/52mΩ/1.4W, U1 STG3856QTR, U2 MCP73831, U3 ESD Diode, U4 AP7347DQ-33W5-7K-3.3V, U5 AP7361C-33

Commit message: Changes resistor divider jumper name and qwiic_led jumper name
Parts:
- renumbered QW_PWR_LED to QWIIC_LED, VIN_REMOVE to DIVIDER
Changed lines of the file:
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@@
 <element name="U$32" library="top" package="CS17" value="" x="99.822" y="7.366" smashed="yes"/>
 <element name="U$25" library="top" package="SWD6522" value="" x="118.872" y="12.7" smashed="yes" rot="R90"/>
-<element name="VIN_REMOVE" library="SparkFun-Jumpers" package="SMT-JUMPER_2_NC_TRACE_SILK" package3d_urn="urn:adsk.eagle:package:39281/1" value="JUMPER-SMT_2_NC_TRACE_SILK" x="114.046" y="22.606" smashed="yes" rot="MR270">
+<element name="DIVIDER" library="SparkFun-Jumpers" package="SMT-JUMPER_2_NC_TRACE_SILK" package3d_urn="urn:adsk.eagle:package:39281/1" value="JUMPER-SMT_2_NC_TRACE_SILK" x="114.046" y="22.606" smashed="yes" rot="MR270">
 <attribute name="NAME" x="112.903" y="22.606" size="0.6096" layer="26" font="vector" ratio="20" rot="MR270" align="bottom-center"/>
 <attribute name="VALUE" x="115.189" y="22.606" size="0.6096" layer="28" font="vector" ratio="20" rot="MR270" align="top-center"/>
@@
 <attribute name="VALUE" x="119.38" y="41.386" size="0.6096" layer="27" font="vector" ratio="20" rot="R180" align="top-center"/>
 </element>
-<element name="QW_PWR_LED" library="SparkFun-Jumpers" package="SMT-JUMPER_2_NC_TRACE_SILK" package3d_urn="urn:adsk.eagle:package:39281/1" value="JUMPER-SMT_2_NC_TRACE_SILK" x="121.793" y="41.91" smashed="yes" rot="MR90">
+<element name="QWIIC_LED" library="SparkFun-Jumpers" package="SMT-JUMPER_2_NC_TRACE_SILK" package3d_urn="urn:adsk.eagle:package:39281/1" value="JUMPER-SMT_2_NC_TRACE_SILK" x="121.793" y="41.91" smashed="yes" rot="MR90">
 <attribute name="NAME" x="122.936" y="41.91" size="0.6096" layer="26" font="vector" ratio="20" rot="MR90" align="bottom-center"/>
 <attribute name="VALUE" x="120.65" y="41.91" size="0.6096" layer="28" font="vector" ratio="20" rot="MR90" align="top-center"/>
@@
 <via x="10.16" y="57.15" extent="1-16" drill="0.3048"/>
 <via x="10.16" y="66.04" extent="1-16" drill="0.3048"/>
-<contactref element="VIN_REMOVE" pad="1"/>
-<contactref element="QW_PWR_LED" pad="1"/>
+<contactref element="DIVIDER" pad="1"/>
+<contactref element="QWIIC_LED" pad="1"/>
 <contactref element="C6" pad="2"/>
 <contactref element="R17" pad="1"/>
@@
 </signal>
 <signal name="N$7">
-<contactref element="VIN_REMOVE" pad="2"/>
+<contactref element="DIVIDER" pad="2"/>
 <contactref element="R7" pad="1"/>
 <wire x1="113.88" y1="20.828" x2="112.903" y2="21.805" width="0.2032" layer="1"/>
@@
 </signal>
 <signal name="N$8">
-<contactref element="QW_PWR_LED" pad="2"/>
+<contactref element="QWIIC_LED" pad="2"/>
 <contactref element="D2" pad="C"/>
 <wire x1="122.936" y1="42.799" x2="122.908" y2="42.827" width="0.2032" layer="1"/>
