File: Hardware/SparkFun_Main_Board_Double_v21.brd (EAGLE design)
At the start: 124.5 x 73.7 mm, 134 parts, among them J1 MICROMOD-2222-C, J10 MICRO-SD-PUSH-PUSH-EXT-PIN, J2 Vertical Qwiic Connector, J4 QWIIC_RIGHT_ANGLE, J5 CORTEX_JTAG_DEBUG_MINIMUM_PTH, J6 MICROMOD_FUNCTION_MAIN, J7 MICROMOD_FUNCTION_MAIN, Q1 3.1A/30V/105mΩ, Q2 20V/4.2A/52mΩ/1.4W, U1 STG3856QTR, U2 MCP73831, U3 ESD Diode, U4 AP7347DQ-33W5-7K-3.3V, U5 AP7361C-33

Commit message: Adds new production files
Parts:
- removed U$3: (no value), top:#PTC#503
- added U$45: (no value), top:#PTC#13
- moved U$17 1.27 mm to (63.5, 48.3)
- moved U$18 1.02 mm to (58.2, 54.5)
Changed lines of the file:
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@@
 <layer number="23" name="tOrigins" color="15" fill="1" visible="yes" active="yes"/>
 <layer number="24" name="bOrigins" color="15" fill="1" visible="yes" active="yes"/>
-<layer number="25" name="tNames" color="7" fill="1" visible="no" active="yes"/>
-<layer number="26" name="bNames" color="7" fill="1" visible="no" active="yes"/>
-<layer number="27" name="tValues" color="7" fill="1" visible="no" active="yes"/>
-<layer number="28" name="bValues" color="7" fill="1" visible="no" active="yes"/>
-<layer number="29" name="tStop" color="7" fill="3" visible="no" active="yes"/>
-<layer number="30" name="bStop" color="7" fill="6" visible="no" active="yes"/>
-<layer number="31" name="tCream" color="7" fill="4" visible="no" active="yes"/>
-<layer number="32" name="bCream" color="7" fill="5" visible="no" active="yes"/>
-<layer number="33" name="tFinish" color="6" fill="3" visible="no" active="yes"/>
-<layer number="34" name="bFinish" color="6" fill="6" visible="no" active="yes"/>
-<layer number="35" name="tGlue" color="7" fill="4" visible="no" active="yes"/>
-<layer number="36" name="bGlue" color="7" fill="5" visible="no" active="yes"/>
-<layer number="37" name="tTest" color="7" fill="1" visible="no" active="yes"/>
-<layer number="38" name="bTest" color="7" fill="1" visible="no" active="yes"/>
+<layer number="25" name="tNames" color="7" fill="1" visible="yes" active="yes"/>
+<layer number="26" name="bNames" color="7" fill="1" visible="yes" active="yes"/>
+<layer number="27" name="tValues" color="7" fill="1" visible="yes" active="yes"/>
+<layer number="28" name="bValues" color="7" fill="1" visible="yes" active="yes"/>
+<layer number="29" name="tStop" color="7" fill="3" visible="yes" active="yes"/>
+<layer number="30" name="bStop" color="7" fill="6" visible="yes" active="yes"/>
+<layer number="31" name="tCream" color="7" fill="4" visible="yes" active="yes"/>
+<layer number="32" name="bCream" color="7" fill="5" visible="yes" active="yes"/>
+<layer number="33" name="tFinish" color="6" fill="3" visible="yes" active="yes"/>
+<layer number="34" name="bFinish" color="6" fill="6" visible="yes" active="yes"/>
+<layer number="35" name="tGlue" color="7" fill="4" visible="yes" active="yes"/>
+<layer number="36" name="bGlue" color="7" fill="5" visible="yes" active="yes"/>
+<layer number="37" name="tTest" color="7" fill="1" visible="yes" active="yes"/>
+<layer number="38" name="bTest" color="7" fill="1" visible="yes" active="yes"/>
 <layer number="39" name="tKeepout" color="4" fill="11" visible="yes" active="yes"/>
-<layer number="40" name="bKeepout" color="1" fill="11" visible="no" active="yes"/>
-<layer number="41" name="tRestrict" color="4" fill="10" visible="no" active="yes"/>
-<layer number="42" name="bRestrict" color="1" fill="10" visible="no" active="yes"/>
-<layer number="43" name="vRestrict" color="2" fill="10" visible="no" active="yes"/>
-<layer number="44" name="Drills" color="7" fill="1" visible="no" active="yes"/>
+<layer number="40" name="bKeepout" color="1" fill="11" visible="yes" active="yes"/>
+<layer number="41" name="tRestrict" color="4" fill="10" visible="yes" active="yes"/>
+<layer number="42" name="bRestrict" color="1" fill="10" visible="yes" active="yes"/>
+<layer number="43" name="vRestrict" color="2" fill="10" visible="yes" active="yes"/>
+<layer number="44" name="Drills" color="7" fill="1" visible="yes" active="yes"/>
 <layer number="45" name="Holes" color="7" fill="1" visible="yes" active="yes"/>
-<layer number="46" name="Milling" color="3" fill="1" visible="no" active="yes"/>
-<layer number="47" name="Measures" color="7" fill="1" visible="no" active="yes"/>
-<layer number="48" name="Document" color="7" fill="1" visible="no" active="yes"/>
+<layer number="46" name="Milling" color="3" fill="1" visible="yes" active="yes"/>
+<layer number="47" name="Measures" color="7" fill="1" visible="yes" active="yes"/>
+<layer number="48" name="Document" color="7" fill="1" visible="yes" active="yes"/>
 <layer number="49" name="Reference" color="13" fill="1" visible="yes" active="yes"/>
-<layer number="50" name="dxf" color="7" fill="1" visible="no" active="yes"/>
+<layer number="50" name="dxf" color="7" fill="1" visible="yes" active="yes"/>
 <layer number="51" name="tDocu" color="6" fill="1" visible="yes" active="yes"/>
-<layer number="52" name="bDocu" color="7" fill="1" visible="no" active="yes"/>
+<layer number="52" name="bDocu" color="7" fill="1" visible="yes" active="yes"/>
 <layer number="91" name="Nets" color="2" fill="1" visible="no" active="no"/>
 <layer number="92" name="Busses" color="1" fill="1" visible="no" active="no"/>
@@
 <element name="U$16" library="top" package="1524" value="" x="23.876" y="16.51" smashed="yes"/>
 <element name="U$13" library="top" package="MAIN523" value="" x="68.58" y="54.61" smashed="yes" rot="MR0"/>
-<element name="U$18" library="top" package="BOARD524" value="" x="57.15" y="54.61" smashed="yes" rot="MR0"/>
+<element name="U$18" library="top" package="BOARD524" value="" x="58.166" y="54.483" smashed="yes" rot="MR0"/>
 <element name="R3" library="SparkFun-Resistors" package="0603" value="2.0k" x="113.411" y="17.907" smashed="yes">
 <attribute name="NAME" x="113.411" y="18.669" size="0.6096" layer="25" font="vector" ratio="20" align="bottom-center"/>
@@
 </element>
 <element name="U$21" library="top" package="MAIN_BOARD5523" value="" x="93.472" y="15.2654" smashed="yes"/>
-<element name="U$17" library="SparkFun-MicroMod" package="MICROMOD_LOGO_1" value="" x="62.23" y="48.26" smashed="yes" rot="MR0"/>
+<element name="U$17" library="SparkFun-MicroMod" package="MICROMOD_LOGO_1" value="" x="63.5" y="48.26" smashed="yes" rot="MR0"/>
 <element name="U$22" library="SparkFun-Aesthetics" package="QWIIC_3MM" value="" x="121.9708" y="54.5592" smashed="yes"/>
 <element name="U$23" library="top" package="STANDOFF501" value="" x="121.8438" y="53.3908" smashed="yes"/>
@@
 <element name="U$38" library="top" package="#EN1_ALT#21" value="" x="78.486" y="8.128" smashed="yes" rot="R90"/>
 <element name="U$27" library="top" package="CHARGE501" value="" x="120.7262" y="6.0198" smashed="yes"/>
-<element name="U$3" library="top" package="#PTC#503" value="" x="121.6152" y="62.5602" smashed="yes" rot="MR0"/>
 <element name="U$7" library="top" package="#SHLD#501" value="" x="112.9792" y="70.0532" smashed="yes" rot="MR0"/>
 <element name="U$30" library="top" package="#I2C#501" value="" x="102.108" y="11.43" smashed="yes" rot="MR0"/>
@@
 <element name="U$43" library="top" package="QWC18" value="" x="123.444" y="42.291" smashed="yes" rot="R90"/>
 <element name="U$44" library="SparkFun-Aesthetics" package="SFE_LOGO_NAME_FLAME_.1" value="" x="43.18" y="2.54" smashed="yes"/>
+<element name="U$45" library="top" package="#PTC#13" value="" x="115.824" y="62.611" smashed="yes" rot="MR0"/>
 </elements>
 <signals>
